File: board/001/001.kicad_pcb (KiCad board)
At the start: 2 copper layers, 50.2 x 50.2 mm, 32 parts, among them T1 BC640, T2 BC640, T3 BC640

Commit message: [UPD] Update unstable CDC version
Routing:
- net S$6: track 10.8 -> 0.00 mm, vias 1 -> 0
- net (no net): track 0.00 -> 7.79 mm
- net S$7: track 10.3 -> 15.2 mm, vias 1 -> 0
